Commit message: remove old templates

File: husky_gazebo/worlds/dock/dock.urdf.xacro (robot description, xacro)
@@ -11,5 +11,5 @@
       <origin xyz="0 0 0" rpy="0 0 0"/>
       <geometry>
-        <mesh filename="package://husky_gazebo/meshes/wibotic/cpr_charge_dock.stl" />
+        <mesh filename="package://husky_gazebo/meshes/cpr_dock_target.stl" />
       </geometry>
     </visual>
@@ -17,5 +17,5 @@
       <origin xyz="0 0 0" rpy="0 0 0"/>
       <geometry>
-        <mesh filename="package://husky_gazebo/meshes/wibotic/cpr_charge_dock.stl" />
+        <mesh filename="package://husky_gazebo/meshes/cpr_dock_target.stl" />
       </geometry>
       <max_contacts>10</max_contacts>
