Commit message: lower lidar to detect dock

File: husky_description/urdf/husky.urdf.xacro (robot description, xacro)
@@ -23,5 +23,5 @@
 <robot name="husky" xmlns:xacro="http://ros.org/wiki/xacro">
   <xacro:arg name="laser_enabled" default="false" />
-  <xacro:arg name="laser_xyz" default="$(optenv HUSKY_LMS1XX_XYZ 0.2206 0.0 0.00635)" />
+  <xacro:arg name="laser_xyz" default="$(optenv HUSKY_LMS1XX_XYZ  0.7 0.0 -0.2)" />
   <xacro:arg name="laser_rpy" default="$(optenv HUSKY_LMS1XX_RPY 0.0 0.0 0.0)" />
   <xacro:arg name="kinect_enabled" default="false" />
@@ -100,4 +100,14 @@
   <gazebo reference="imu_link">
   </gazebo>
+    <!-- GPS Link is the standard mounting position-->
+  <!-- Can be modified with environment variables in /etc/ros/setup.bash -->
+  <link name="gps_link"/>
+  <joint name="gps_joint" type="fixed">
+    <origin xyz="$(optenv HUSKY_GPS_XYZ 0.19 0 0.149)" rpy="$(optenv HUSKY_GPS_RPY 0 -1.5708 3.1416)" />
+    <parent link="base_link" />
+    <child link="gps_link" />
+  </joint>
+  <gazebo reference="gps_link">
+  </gazebo>
   <!-- Husky wheel macros -->
   <xacro:husky_wheel wheel_prefix="front_left">
@@ -158,5 +168,5 @@
       <updateRate>40</updateRate>
       <bodyName>base_link</bodyName>
-      <frameId>base_link</frameId>
+      <frameId>gps_link</frameId>
       <topicName>navsat/fix</topicName>
       <velocityTopicName>navsat/vel</velocityTopicName>

Commit message: rear lidar

File: husky_description/urdf/husky.urdf.xacro (robot description, xacro)
@@ -25,4 +25,7 @@
   <xacro:arg name="laser_xyz" default="$(optenv HUSKY_LMS1XX_XYZ  0.38 0.0 -0.2)" />
   <xacro:arg name="laser_rpy" default="$(optenv HUSKY_LMS1XX_RPY 0.0 0.0 0.0)" />
+  <xacro:arg name="rear_laser_enabled" default="false" />
+  <xacro:arg name="rear_laser_xyz" default="$(optenv HUSKY_LMS1XX_XYZ  -0.58 0.0 -0.2)" />
+  <xacro:arg name="rear_laser_rpy" default="$(optenv HUSKY_LMS1XX_RPY 0.0 0.0 3.1415)" />
   <xacro:arg name="kinect_enabled" default="false" />
   <xacro:arg name="kinect_xyz" default="$(optenv HUSKY_KINECT_XYZ 0 0 0)" />
@@ -133,4 +136,13 @@
     </joint>
   </xacro:if>
+  <xacro:if value="$(arg laser_enabled)">
+    <sick_lms1xx_mount prefix="rear_base"/>
+    <sick_lms1xx frame="rear_base_laser" topic="scan_rear" robot_namespace="$(arg robot_namespace)"/>
+    <joint name="rear_laser_mount_joint" type="fixed">
+      <origin xyz="$(arg rear_laser_xyz)" rpy="$(arg rear_laser_rpy)" />
+      <parent link="top_plate_link" />
+      <child link="rear_base_laser_mount" />
+    </joint>
+  </xacro:if>
   <xacro:if value="$(arg kinect_enabled)">
     <xacro:sensor_arch prefix="" parent="top_plate_link">
@@ -147,4 +159,5 @@
     <plugin name="gazebo_ros_control" filename="libgazebo_ros_control.so">
       <robotNamespace>$(arg robot_namespace)</robotNamespace>
+      <legacyModeNS>true</legacyModeNS>
     </plugin>
   </gazebo>

Commit message: gps issue

File: husky_description/urdf/husky.urdf.xacro (robot description, xacro)
@@ -103,14 +103,4 @@
   <gazebo reference="imu_link">
   </gazebo>
-    <!-- GPS Link is the standard mounting position-->
-  <!-- Can be modified with environment variables in /etc/ros/setup.bash -->
-  <link name="gps_link"/>
-  <joint name="gps_joint" type="fixed">
-    <origin xyz="$(optenv HUSKY_GPS_XYZ 0.19 0 0.149)" rpy="$(optenv HUSKY_GPS_RPY 0 -1.5708 3.1416)" />
-    <parent link="base_link" />
-    <child link="gps_link" />
-  </joint>
-  <gazebo reference="gps_link">
-  </gazebo>
   <!-- Husky wheel macros -->
   <xacro:husky_wheel wheel_prefix="front_left">
@@ -181,10 +171,10 @@
       <updateRate>40</updateRate>
       <bodyName>base_link</bodyName>
-      <frameId>gps_link</frameId>
+      <frameId>base_link</frameId>
       <topicName>navsat/fix</topicName>
       <velocityTopicName>navsat/vel</velocityTopicName>
       <referenceLatitude>43.50076203</referenceLatitude>
       <referenceLongitude>-80.54629721</referenceLongitude>
-      <referenceHeading>0</referenceHeading>
+      <referenceHeading>90.0</referenceHeading>
       <referenceAltitude>0</referenceAltitude>
       <drift>0.0001 0.0001 0.0001</drift>

Commit message: dock testingn for HITT01

File: husky_description/urdf/husky.urdf.xacro (robot description, xacro)
@@ -25,9 +25,8 @@
   <xacro:arg name="laser_xyz" default="$(optenv HUSKY_LMS1XX_XYZ  0.2206 0.0 0.00635)" />
   <xacro:arg name="laser_rpy" default="$(optenv HUSKY_LMS1XX_RPY 0.0 0.0 0.0)" />
--->
+<!--   <xacro:arg name="laser_enabled" default="false" />
+  <xacro:arg name="laser_xyz" default="$(optenv HUSKY_LMS1XX_XYZ  0.38 0.0 -0.25)" />
+  <xacro:arg name="laser_rpy" default="$(optenv HUSKY_LMS1XX_RPY 0.0 0.0 0.0)" /> -->
 <!--
-  <xacro:arg name="laser_enabled" default="false" />
-  <xacro:arg name="laser_xyz" default="$(optenv HUSKY_LMS1XX_XYZ  0.38 0.0 -0.2)" />
-  <xacro:arg name="laser_rpy" default="$(optenv HUSKY_LMS1XX_RPY 0.0 0.0 0.0)" />
   <xacro:arg name="rear_laser_enabled" default="false" />
   <xacro:arg name="rear_laser_xyz" default="$(optenv HUSKY_LMS1XX_XYZ  -0.58 0.0 -0.2)" />

File: husky_gazebo/worlds/dock/dock.urdf.xacro (robot description, xacro)
@@ -11,5 +11,5 @@
       <origin xyz="0 0 0" rpy="0 0 0"/>
       <geometry>
-        <mesh filename="package://husky_gazebo/meshes/cpr_dock_target.stl" />
+        <mesh filename="package://husky_gazebo/meshes/Dock_X5.stl" scale="0.001 0.001 0.001"/>
       </geometry>
     </visual>
@@ -17,5 +17,5 @@
       <origin xyz="0 0 0" rpy="0 0 0"/>
       <geometry>
-        <mesh filename="package://husky_gazebo/meshes/cpr_dock_target.stl" />
+        <mesh filename="package://husky_gazebo/meshes/Dock_X5.stl" scale="0.001 0.001 0.001"/>
       </geometry>
       <max_contacts>10</max_contacts>
@@ -35,5 +35,5 @@
   </link>
   <gazebo reference="base_link">
-    <material>Gazebo/DarkGray</material>
+    <material>Gazebo/Yellow</material>
   </gazebo>
   <gazebo> <static>true</static></gazebo>
